File: ENTRENADOR_SMD/ENTRENADOR_SMD.sch (EAGLE design)
At the start: 76 parts, among them IC1 PIC16F1939PT, SW1 TL3342F160QG/TR

Commit message: Se actualiza y se argegan librerias
Parts:
- added IC2: 7824T, linear:7824T
- added J1: DCJ0202, con-jack:DCJ0202
- added U$1, U$2, U$4, U$5: CAPA, CAPAE830X1000N:CAPA
- added U$3: VREG3V3, VREG_L7805ACD2T:VREG3V3
- added X1: (no value), con-ptr500:AK300/2
- renumbered JP1 to POT, JP2 to JP_5V5, JP3 to JP_3V3, JP4 to SOC_UART, JP5 to JP_I2C, LEDS3 to BTN_A, LEDS4 to BTN_B, S2 to PWR_SLIDE
Connections:
- removed net GNG: PD-9.KL
- new net N$36: IC2.VI, J1.1, U$4.P, X1-1.KL
- net 3V3: now also U$2.P, U$3.OUT
- net GND: now also IC2.GND, J1.2, J1.3, PD-9.KL, U$1.N, U$2.N, U$3.GND, U$4.N, U$5.N, X1-2.KL
- net VCC: now also U$1.P, U$3.IN
- net VEXT: now also IC2.VO, U$5.P
Other:
- moved on the sheet: R19

Commit message: se crea diseño entrenador
Parts:
- removed JP_SLIDES1, JP_SLIDES2: (no value), pinhead:PINHD-1X4
- added JP_SLIDES_DOWN, JP_SLIDES_UP: (no value), pinhead:PINHD-1X4
- added R23, R24, R25, R26, R27, R28, R29, R30: 4K7, R0805_:R-EU_R0805
- R1: value (none) -> 4K7
- R10, R11, R12, R13, R14, R15, R16, R17: value (none) -> 10K
- R19, R20, R21: value 3386P-1-101TLF -> COM-09806; device 3386P-1-101TLF:3386P-1-101TLF -> COM-09806:COM-09806
- R2, R3, R4, R5, R6, R7, R8, R9: value (none) -> 330R
- renumbered LED1 to L1, LED4 to L4, LED5 to L5, LED8 to L8
Connections:
- new net N$37: JP_SLIDES_UP.1, R27.1
- new net N$38: JP_SLIDES_UP.2, R28.1
- new net N$39: JP_SLIDES_UP.3, R29.1
- new net N$40: JP_SLIDES_DOWN.1, R26.1
- new net N$41: JP_SLIDES_DOWN.2, R25.1
- new net N$42: JP_SLIDES_DOWN.3, R24.1
- new net N$43: JP_SLIDES_DOWN.4, R23.1
- new net N$44: JP_SLIDES_UP.4, R30.1
- net N$1: now also R23.2; no longer JP_SLIDES1.4
- net N$2: now also R24.2; no longer JP_SLIDES1.3
- net N$3: now also R25.2; no longer JP_SLIDES1.2
- net N$4: now also R26.2; no longer JP_SLIDES1.1
- net N$5: now also R30.2; no longer JP_SLIDES2.4
- net N$6: now also R29.2; no longer JP_SLIDES2.3
- net N$7: now also R28.2; no longer JP_SLIDES2.2
- net N$8: now also R27.2; no longer JP_SLIDES2.1
