File: COPIA ENTRENADOR/Entrenadorv01.sch (EAGLE design)
At the start: 63 parts, among them IC1 7805T, X1 MINI-USB_4P-85-32004-10X

Commit message: se agrega diseño PCB
Parts:
- added BAT1: (no value), sn2032:SN2032
- added C5, C6: (no value), rcl:C-EU025-025X050
- added CON_LCD, DATOS_7_SEG, LEDS, PORTA, PORTB, PORTC, PORTD, TECLADO: 2510-, con-3m:2510-
- added DIS1, DIS2: HD-K123, display-hp:HD-K123
- added DS1307: DS1307, ds1307_pcf8583:DS1307
- added EEPROM: 24LC256P, microchip:24LC256P
- added FUENTE_ULN: (no value), con-ptr500:AK300/2
- added I2C_16F, I2C_18F, MOD_I2C: (no value), pinhead:PINHD-1X2
- added IC5: (no value), uln-udn:ULN2803A
- added JP2: (no value), pinhead:PINHD-1X4
- added JP6: (no value), pinhead:PINHD-1X3
- added JP7: (no value), pinhead:PINHD-1X8
- added JUMP_LCD, SALIDAS_ULN: (no value), pinhead:PINHD-1X6
- added K3, K4: SRD-05VDC-SL-C, SRD-05VDC-SL-C (1):SRD-05VDC-SL-C
- added LS1: CST-951AP, CST-951AP:CST-951AP
- added Q2: (no value), special:XTAL/S
- added R15, R16, R29, R30, R31, R32, R35, R36: 10K, rcl:R-EU_0207/10
- added R17, R18, R21, R22, R25, R26, R27, R33, R34: 330, rcl:R-EU_0207/10
- added R28, R37, R38, R39: 5K, rcl:R-TRIMM3339P
- added R40, R41, R42: 10k, rcl:R-EU_0207/10
- added RELAY_1, RELAY_2: (no value), con-ptr500:AK300/3
- added S4: (no value), switch:M251
- added T1, T2, T3, T4: 2N3904, transistor:2N3904
- added U$1: LCD-HD4478020X4-3HOLES, HD44780LCD:LCD-HD4478020X4-3HOLES
- added U$2: (no value), keypad_4x4_raw:KEYPAD4X4
Connections:
- new net A: DIS1.A1, DIS1.A2, DIS2.A1, DIS2.A2, R34.1
- new net B: DIS1.B1, DIS1.B2, DIS2.B1, DIS2.B2, R33.1
- new net C: DIS1.C1, DIS1.C2, DIS2.C1, DIS2.C2, R26.1
- new net D: DIS1.D1, DIS1.D2, DIS2.D1, DIS2.D2, R25.1
- new net E: DIS1.E1, DIS1.E2, DIS2.E1, DIS2.E2, R22.1
- new net F: DIS1.F1, DIS1.F2, DIS2.F1, DIS2.F2, R21.1
- new net G: DIS1.G1, DIS1.G2, DIS2.G1, DIS2.G2, R18.1
- new net N$10: JP6.2, R38.S
- new net N$100: FUENTE_ULN-2.KL, IC5.CD+, K3.A1, K4.A1, LS1.P
- new net N$101: R28.A, S4.O, U$1.A, U$1.VDD
- new net N$12: JP6.3, R37.S
- new net N$13: R27.1, U$1.K
- new net N$14: JP6.1, R39.S
- new net N$15: IC5.I1, JP7.1
- new net N$18: CON_LCD-8.KL, JUMP_LCD.6, U$1.DB7
- new net N$19: CON_LCD-7.KL, JUMP_LCD.5, U$1.DB6
- new net N$20: IC5.I2, JP7.2
- new net N$21: CON_LCD-6.KL, JUMP_LCD.4, U$1.DB5
- new net N$22: DS1307.SCL, EEPROM.SCL, MOD_I2C.1, R40.2
- new net N$23: CON_LCD-5.KL, JUMP_LCD.3, U$1.DB4
- new net N$24: IC5.I3, JP7.3
- new net N$25: CON_LCD-1.KL, JUMP_LCD.1, U$1.RS
- new net N$26: DIS1.DP1, DIS1.DP2, DIS2.DP1, DIS2.DP2, R17.2
- new net N$27: CON_LCD-2.KL, JUMP_LCD.2, U$1.E
- new net N$28: R30.1, TECLADO-1.KL, U$2.C1
- new net N$29: R28.S, U$1.VO
- new net N$30: R29.1, TECLADO-2.KL, U$2.C2
- new net N$31: R31.1, TECLADO-3.KL, U$2.C3
- new net N$32: R32.1, TECLADO-4.KL, U$2.C4
- new net N$33: TECLADO-5.KL, U$2.R1
- new net N$34: TECLADO-6.KL, U$2.R2
- new net N$35: TECLADO-7.KL, U$2.R3
- new net N$36: TECLADO-8.KL, U$2.R4
- new net N$37: DATOS_7_SEG-7.KL, R18.2
- new net N$38: R16.1, T1.B
- new net N$40: R15.1, T2.B
- new net N$41: DIS1.CC2, T2.E
- new net N$42: DIS1.CC1, T1.E
- new net N$59: DATOS_7_SEG-6.KL, R21.2
- new net N$60: JP2.1, R16.2
- new net N$61: JP2.2, R15.2
- new net N$62: DATOS_7_SEG-5.KL, R22.2
- new net N$63: DATOS_7_SEG-4.KL, R25.2
- new net N$64: DATOS_7_SEG-3.KL, R26.2
- new net N$65: DATOS_7_SEG-2.KL, R33.2
- new net N$66: DATOS_7_SEG-1.KL, R34.2
- new net N$67: DATOS_7_SEG-8.KL, R17.1
- new net N$68: R35.1, T3.B
- new net N$70: R36.1, T4.B
- new net N$71: JP2.4, R36.2
- new net N$72: JP2.3, R35.2
- new net N$73: DIS2.CC1, T3.E
- new net N$74: DIS2.CC2, T4.E
- new net N$75: IC5.I4, JP7.4
- new net N$76: IC5.I5, JP7.5
- new net N$77: BAT1.+, DS1307.VBAT
- new net N$78: DS1307.SQW, R42.2
- new net N$79: IC5.I6, JP7.6
- new net N$80: DS1307.SDA, EEPROM.SDA, MOD_I2C.2, R41.2
- new net N$81: C5.1, DS1307.X1, Q2.2
- new net N$82: C6.1, DS1307.X2, Q2.1
- new net N$83: IC5.I7, JP7.7
- new net N$84: IC5.I8, JP7.8
- new net N$85: IC5.O8, LS1.M
- new net N$86: IC5.O1, K3.A2
- new net N$87: K3.COM, RELAY_1-2.KL
- new net N$88: IC5.O5, SALIDAS_ULN.3
- new net N$89: IC5.O2, K4.A2
- new net N$90: IC5.O3, SALIDAS_ULN.1
- new net N$91: IC5.O4, SALIDAS_ULN.2
- new net N$92: IC5.O6, SALIDAS_ULN.4
- new net N$93: IC5.O7, SALIDAS_ULN.5
- new net N$94: K3.NO, RELAY_1-3.KL
- new net N$95: K3.NC, RELAY_1-1.KL
- new net N$96: K4.NO, RELAY_2-3.KL
- new net N$97: K4.COM, RELAY_2-2.KL
- new net N$98: K4.NC, RELAY_2-1.KL
- net AUX_B6: now also PORTB-7.KL
- net AUX_B7: now also PORTB-8.KL
- net GND: now also BAT1.-, C5.2, C6.2, CON_LCD-10.KL, DS1307.GND, EEPROM.A0, EEPROM.A1, EEPROM.A2, EEPROM.GND, EEPROM.WP, FUENTE_ULN-1.KL, IC5.GND, LEDS-10.KL, PORTA-10.KL, PORTB-10.KL, PORTC-10.KL, PORTD-10.KL, R27.2, R28.E, R29.2, R30.2, R31.2, R32.2, R37.A, R38.A, R39.A, SALIDAS_ULN.6, TECLADO-10.KL, U$1.DB0, U$1.DB1, U$1.DB2, U$1.DB3, U$1.R/W, U$1.VSS
- net N$51: now also LEDS-1.KL
- net N$52: now also LEDS-2.KL
- net N$53: now also LEDS-3.KL
- net N$54: now also LEDS-4.KL
- net N$55: now also LEDS-5.KL
- net N$56: now also LEDS-6.KL
- net N$57: now also LEDS-7.KL
- net N$58: now also LEDS-8.KL
- net RA0: now also PORTA-1.KL
- net RA1: now also PORTA-2.KL
- net RA2: now also PORTA-3.KL
- net RA3: now also PORTA-4.KL
- net RA4: now also PORTA-5.KL
- net RA5: now also PORTA-6.KL
- net RB0: now also I2C_18F.1, PORTB-1.KL
- net RB1: now also I2C_18F.2, PORTB-2.KL
- net RB2: now also PORTB-3.KL
- net RB3: now also PORTB-4.KL
- net RB4: now also PORTB-5.KL
- net RB5: now also PORTB-6.KL
- net RC0: now also PORTC-1.KL
- net RC1: now also PORTC-2.KL
- net RC2: now also PORTC-3.KL
- net RC3: now also I2C_16F.1, PORTC-4.KL
- net RC4: now also I2C_16F.2, PORTC-5.KL
- net RC5: now also PORTC-6.KL
- net RC6: now also PORTC-7.KL
- net RC7: now also PORTC-8.KL
- net RD0: now also PORTD-1.KL
- net RD1: now also PORTD-2.KL
- net RD2: now also PORTD-3.KL
- net RD3: now also PORTD-4.KL
- net RD4: now also PORTD-5.KL
- net RD5: now also PORTD-6.KL
- net RD6: now also PORTD-7.KL
- net RD7: now also PORTD-8.KL
- net VCC: now also CON_LCD-9.KL, DS1307.VCC, EEPROM.VCC, LEDS-9.KL, PORTA-9.KL, PORTB-9.KL, PORTC-9.KL, PORTD-9.KL, R37.E, R38.E, R39.E, R40.1, R41.1, R42.1, S4.P, T1.C, T2.C, T3.C, T4.C, TECLADO-9.KL
Other:
- note added: "DISPLAY 7 SEGMENTOS"
- note added: "INTERFACE I2C"
- note added: "KEYPAD 4x4"
- note added: "LCD 4x20"
- note added: "POTS ADC"
- note added: "SALIDAS DE 500mA"
